File: side.kicad_sch (KiCad schematic)
At the start: 70 parts, among them SW1 SW_Push, SW10 SW_Push, SW13 SW_Push, SW14 SW_Push, SW15 SW_Push, SW16 SW_Push, SW17 SW_Push, SW18 SW_Push, SW25 SW_Push, SW26 SW_Push, SW27 SW_Push, SW28 SW_Push, SW29 SW_Push, SW3 SW_Push, SW30 SW_Push, SW37 SW_Push, SW38 SW_Push, SW39 SW_Push, SW40 SW_Push, SW41 SW_Push, SW42 SW_Push, SW49 SW_Push, SW5 SW_Push, SW50 SW_Push, SW51 SW_Push, SW55 SW_Push, SW57 RotaryEncoder_Switch_MP, SW6 SW_Push, SW9 SW_Push, U1 Seeeduino Xiao nRF52840, U3 MCP23017_SO, U7 MCP1700x-330xxTT

Commit message: more stuff
Connections:
- net UnderKeyLED/DIN12: no longer names the net of U3.7 (GPB6)
Other:
- removed sheet UnderKeyLED
Changed lines of the file:
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@@
 	(wire
 		(pts
-			(xy 97.79 48.26) (xy 97.79 157.48)
-		)
-		(stroke
-			(width 0)
-			(type default)
-		)
-	)
-	(wire
-		(pts
 			(xy 205.74 100.33) (xy 223.52 100.33)
 		)
@@
 	(wire
 		(pts
-			(xy 97.79 157.48) (xy 76.2 157.48)
-		)
-		(stroke
-			(width 0)
-			(type default)
-		)
-	)
-	(wire
-		(pts
 			(xy 189.23 115.57) (xy 205.74 115.57)
 		)
@@
 	(wire
 		(pts
-			(xy 266.7 48.26) (xy 97.79 48.26)
-		)
-		(stroke
-			(width 0)
-			(type default)
-		)
-	)
-	(wire
-		(pts
 			(xy 142.24 163.83) (xy 142.24 151.13)
 		)
@@
 	(wire
 		(pts
-			(xy 266.7 63.5) (xy 266.7 48.26)
-		)
-		(stroke
-			(width 0)
-			(type default)
-		)
-	)
-	(wire
-		(pts
 			(xy 125.73 53.34) (xy 125.73 63.5)
 		)
@@
 				)
 			)
-		)
-	)
-	(sheet
-		(at 241.3 63.5)
-		(size 38.1 52.07)
-		(exclude_from_sim no)
-		(in_bom yes)
-		(on_board yes)
-		(dnp no)
-		(fields_autoplaced yes)
-		(stroke
-			(width 0.1524)
-			(type solid)
-		)
-		(fill
-			(color 0 0 0 0.0000)
-		)
-		(property "Sheetname" "UnderKeyLED"
-			(at 241.3 62.7884 0)
-			(effects
-				(font
-					(size 1.27 1.27)
-				)
-				(justify left bottom)
-			)
-		)
-		(property "Sheetfile" "underkeyled.kicad_sch"
-			(at 241.3 116.1546 0)
-			(effects
-				(font
-					(size 1.27 1.27)
-				)
-				(justify left top)
-			)
-		)
-		(pin "DIN12" input
-			(at 266.7 63.5 90)
-			(effects
-				(font
-					(size 1.27 1.27)
-				)
-				(justify right)
-			)
-		)
-		(instances
-			(project "SplitCodeBoard"
-				(path "/8e037d1a-38ef-4c72-8142-d24fba09340a/212c55d9-bd52-4ba0-a9c1-1485280a605d"
-					(page "4")
-				)
-			)
