File: SplitCodeBoard.kicad_pcb (KiCad board)
At the start: 2 copper layers, 318.3 x 127 mm, 208 parts, among them SW1 SW_Push, SW10 SW_Push, SW11 SW_Push, SW12 SW_Push, SW13 SW_Push, SW14 SW_Push, SW15 SW_Push, SW16 SW_Push, SW17 SW_Push, SW18 SW_Push, SW19 SW_Push, SW2 SW_Push, SW20 SW_Push, SW21 SW_Push, SW22 SW_Push, SW23 SW_Push, SW24 SW_Push, SW25 SW_Push, SW26 SW_Push, SW27 SW_Push, SW28 SW_Push, SW29 SW_Push, SW3 SW_Push, SW30 SW_Push, SW31 SW_Push, SW32 SW_Push, SW33 SW_Push, SW34 SW_Push, SW35 SW_Push, SW36 SW_Push, SW37 SW_Push, SW38 SW_Push, SW39 SW_Push, SW4 SW_Push, SW40 SW_Push, SW41 SW_Push, SW42 SW_Push, SW43 SW_Push, SW44 SW_Push, SW45 SW_Push, SW46 SW_Push, SW47 SW_Push, SW48 SW_Push, SW49 SW_Push, SW5 SW_Push, SW50 SW_Push, SW51 SW_Push, SW52 SW_Push, SW53 SW_Push, SW54 SW_Push, SW55 SW_Push, SW56 SW_Push, SW58 RotaryEncoder_Switch_MP, SW6 SW_Push, SW7 SW_Push, SW8 SW_Push, SW9 SW_Push, U1 Seeeduino Xiao nRF52840, U2 Seeeduino Xiao nRF52840, U3 MCP23017_SO, U4 MCP23017_SO, U7 MCP1700x-330xxTT, U8 MCP1700x-330xxTT

Commit message: more stuff
Parts:
- removed D100, D101, D102, D103, D104, D105, D106, D107, D108, D109, D110, D111, D112, D113, D114, D115, D116, D121, D122, D123, D124, D71, D72, D73, D74, D75, D76, D77, D78, D79, D80, D81, D82, D83, D84, D85, D86, D87, D88, D89, D90, D91, D92, D93, D94, D95, D96, D97, D98, D99: SK6812MINI, LED_SMD:LED_SK6812MINI_PLCC4_3.5x3.5mm_P1.75mm
- added H1: MountingHole, Panelization:MouseBite-Slot_2.0x2.0mm_inset_D0.5mm_P0.85mm_4h_Trace, F.Cu at (191.0, 129.5)
- added H1: MountingHole, Panelization:MouseBite-Slot_2.0x2.0mm_inset_D0.5mm_P0.85mm_4h_Trace, F.Cu at (226.0, 129.5)
- added H1: MountingHole, Panelization:MouseBite-Slot_2.0x2.0mm_inset_D0.5mm_P0.85mm_4h_Trace, F.Cu at (209.0, 129.5)
- added J1: OLED, KiCad-SSD1306-0.91-OLED-4pin-128x32:SSD1306-0.91-OLED-4pin-128x32, B.Cu at (205.0, 86.7)
- added R7: R, Resistor_SMD:R_0201_0603Metric, B.Cu at (185.8, 90.2)
- added R8: R, Resistor_SMD:R_0201_0603Metric, B.Cu at (185.8, 92.0)
- added SW59: SW_Push, PCM_marbastlib-choc:SW_choc_v1_HS_CPG135001S30_1u, F.Cu at (207.3, 97.0)
- added SW60: SW_Push, PCM_marbastlib-choc:SW_choc_v1_HS_CPG135001S30_1u, F.Cu at (223.7, 97.0)
- added SW61: SW_Push, PCM_marbastlib-choc:SW_choc_v1_HS_CPG135001S30_1u, F.Cu at (240.0, 97.0)
- added SW62: SW_Push, PCM_marbastlib-choc:SW_choc_v1_HS_CPG135001S30_1u, F.Cu at (207.7, 116.5)
- added SW63: SW_Push, PCM_marbastlib-choc:SW_choc_v1_HS_CPG135001S30_1u, F.Cu at (224.0, 116.5)
- added SW64: SW_Push, PCM_marbastlib-choc:SW_choc_v1_HS_CPG135001S30_1u, F.Cu at (240.4, 116.5)
- added TP5: BAT, TestPoint:TestPoint_Pad_2.0x2.0mm, B.Cu at (189.0, 87.0)
- added TP6: GND, TestPoint:TestPoint_Pad_2.0x2.0mm, B.Cu at (189.0, 91.0)
- added U10: ~, TP4056:TP4056-18650, F.Cu at (195.9, 74.8)
- added U11: MCP1700x-330xxTT, Package_TO_SOT_SMD:SOT-23, B.Cu at (184.5, 87.2)
- added U9: Seeeduino Xiao nRF52840, PCM_marbastlib-xp-promicroish:Xiao_nRF52840_ACH, B.Cu at (187.8, 113.4)
- D57, D58, D59, D60, D61, D62, D63, D64, SW58: moved to B.Cu
- D65, D66, D67, D68, D69, D70: value SK6812MINI -> D; footprint LED_SMD:LED_SK6812MINI_PLCC4_3.5x3.5mm_P1.75mm -> Diode_SMD:D_SOD-123
- moved D67 140.8 mm to (246.0, 101.3), turned to 90 degrees
- moved D65 131.8 mm to (213.0, 101.7), turned to 90 degrees
- moved D66 107.3 mm to (229.5, 101.7), turned to 90 degrees
- moved D69 105.8 mm to (229.5, 121.3), turned to 90 degrees
- moved D68 104.3 mm to (213.5, 121.3), turned to 90 degrees
- moved D70 101.3 mm to (246.0, 121.3), turned to 90 degrees
- moved D63 59.8 mm to (62.2, 175.6)
- moved D61 47.0 mm to (62.2, 168.0)
- moved SW58 43.4 mm to (364.5, 145.0), turned to 180 degrees
- moved SW17 40.5 mm to (169.1, 157.8)
- moved SW18 40.5 mm to (190.1, 161.0)
- moved SW29 40.5 mm to (169.1, 179.3)
- moved SW30 40.5 mm to (190.1, 182.5)
- moved D19 40.5 mm to (233.2, 165.1)
- moved D31 40.5 mm to (233.7, 186.6)
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Connections:
- D65 pad 1: Net-(D65-DOUT) -> /ROW1
- D65 pad 2: GND -> Net-(D65-A)
- D66 pad 1: Net-(D66-DOUT) -> /ROW1
- D66 pad 2: GND -> Net-(D66-A)
- D67 pad 1: Net-(D67-DOUT) -> /ROW1
- D67 pad 2: GND -> Net-(D67-A)
- D68 pad 1: Net-(D68-DOUT) -> /ROW2
- D68 pad 2: GND -> Net-(D68-A)
- D69 pad 1: Net-(D69-DOUT) -> /ROW2
- D69 pad 2: GND -> Net-(D69-A)
- D70 pad 1: Net-(D70-DOUT) -> /ROW2
- D70 pad 2: GND -> Net-(D70-A)
- U3 pad 7: /left/UnderKeyLED/DIN12 -> unconnected-(U3-GPB6-Pad7)
- U4 pad 7: /right/UnderKeyLED/DIN12 -> unconnected-(U4-GPB6-Pad7)
Routing:
- net +5V: track 1804.3 -> 339.8 mm, vias 68 -> 1
- net GND: track 2162.4 -> 1504.8 mm, vias 45 -> 40
- net /COL3: track 0.00 -> 132.2 mm
- net Net-(J1-Pin_3): track 0.00 -> 81.9 mm
- net Net-(J1-Pin_4): track 0.00 -> 81.6 mm
- net /left/UnderKeyLED/DIN12: track 76.2 -> 0.00 mm, vias 1 -> 0
- net Net-(D104-DOUT): track 70.7 -> 0.00 mm, vias 2 -> 0
- net /ROW1: track 0.00 -> 70.1 mm
- net /ROW2: track 0.00 -> 68.7 mm
- net /right/UnderKeyLED/DIN12: track 64.3 -> 0.00 mm, vias 1 -> 0
- net /COL2: track 0.00 -> 57.4 mm, vias 0 -> 3
- net Net-(D67-DOUT): track 44.5 -> 0.00 mm
- net Net-(D73-DOUT): track 44.3 -> 0.00 mm
- net Net-(D69-DOUT): track 43.2 -> 0.00 mm
- net Net-(D70-DOUT): track 40.4 -> 0.00 mm
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Other:
- board size 318.3 x 127 mm -> 318.3 x 177 mm

Commit message: Added Case
Parts:
- added ?: LOGO, LOGO, B.Cu at (232.0, 220.8)
- added ?: LOGO, LOGO, B.Cu at (280.9, 209.9)
- added ?: LOGO, LOGO, B.Cu at (212.2, 169.1)
- added ?: LOGO, LOGO, B.Cu at (114.5, 215.0)
- added ?: LOGO, LOGO, B.Cu at (134.5, 215.0)
- added G***: LOGO, LOGO, F.Cu at (231.0, 76.4)
- added G***: LOGO, LOGO, F.Cu at (58.0, 168.5)
- added G***: LOGO, LOGO, F.Cu at (210.0, 175.6)
- added G***: LOGO, LOGO, F.Cu at (356.8, 179.3)
- added G***: LOGO, LOGO, F.Cu at (208.4, 196.8)
- added G***: LOGO, LOGO, F.Cu at (209.8, 75.6)
- added G***: LOGO, LOGO, B.Cu at (209.0, 147.3)
- QR${REFERENCE}: moved to F.Cu
- moved QR${REFERENCE} 162.1 mm to (232.0, 83.5), turned to 0 degrees
Connections:
- U9 pad 1: unconnected-(U9-P0.02-Pad1) -> /BT_PIN
- U9 pad 14: /BT_PIN -> unconnected-(U9-P1.12-Pad14)
Routing:
- net /BT_PIN: track 37.5 -> 41.9 mm, vias 0 -> 1
Other:
- board text added: "By Ruben Sutton Github: @code2344/SplitCodeBoard made for Stasis"
- board text added: "HELLO FROM THE BACK OF THE PCB IF YOU ARE READING THIS YOU SHOULD PROBABLY FLIP THE BOARD"
- board text added: "Left SplitCodeBoard v1"
- board text added: "Right SplitCodeBoard v1"
- board text added: "SplitCodeBoard v1.0"
- board text added: "SplitCodeBoard v1.0 A project for Hack Club Stasis Made in Tasmania by Ruben S Github: @code2344/SplitCodeBoard Find me at https://scstudios.tech"
- board text added: "THIS WAY IS UP --------------------------->"
- board text added: "THIS WAY IS UP ------------------------->"
- board text added: "THIS WAY UP ------------------------------>"
- board text added: "this is the back of the pcb :)"
- board text removed: "Left Keyboard"
